File: Hardware/BivalveBit_main_board_KiCAD/BivalveBit_RevE/BivalveBit.kicad_pcb (KiCad board)
At the start: 2 copper layers, 89.9 x 17.8 mm, 58 parts, among them J2 Conn_01x01_Male, J4 Conn_01x01_Male, J5 Conn_01x01_Male, J6 Conn_01x03_Male, J7 Conn_01x01_Male, J8 Conn_01x01_Male, Q1 BSS138, Q2 BSS138, Q3 P-FET, SW2 SW_Reed, U2 ATmega4808-A, U3 LP5907MFX-3.0, U4 BJT_NPN

Commit message: Saving some layout images
Other:
- net class Default removed
