File: Hardware/BivalveBit_main_board_KiCAD/BivalveBit_RevF/BivalveBit_RevF.kicad_pcb (KiCad board)
At the start: 2 copper layers, 89.9 x 17.8 mm, 59 parts, among them J4 Conn_01x01_Male, J5 Conn_01x01_Male, J6 Conn_01x03_Male, J7 Conn_01x01_Male, J8 Conn_01x01_Male, Q1 BSS138, Q2 BSS138, Q3 P-FET, SW2 SW_Reed, U2 ATmega4808-A, U3 LP5907MFX-3.0, U4 BJT_NPN

Commit message: Few minor label changes
Other:
- board text added: "BivalveBit RevF 2024 luke.miller@sdsu.edu"
- board text removed: "BivalveBit RevF 2023 luke.miller@sdsu.edu"
Changed lines of the file:
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@@
     (effects (font (size 0.7112 0.7112) (thickness 0.127)) (justify mirror))
   )
-  (gr_text "+" (at 109.4359 130.8862 180) (layer "B.SilkS")
+  (gr_text "+" (at 109.84 128.222 180) (layer "B.SilkS")
     (effects (font (size 0.7112 0.7112) (thickness 0.127)) (justify mirror))
   )
-  (gr_text "GND" (at 109.5121 132.7658 270) (layer "B.SilkS")
+  (gr_text "GND" (at 110.2 130.482 270) (layer "B.SilkS")
     (effects (font (size 0.7112 0.7112) (thickness 0.127)) (justify mirror))
   )
@@
     (effects (font (size 1.016 1.016) (thickness 0.1524)) (justify mirror))
   )
-  (gr_text "BivalveBit RevF 2023\nluke.miller@sdsu.edu" (at 119.6467 122.4915) (layer "B.SilkS")
+  (gr_text "BivalveBit RevF 2024\nluke.miller@sdsu.edu" (at 119.6467 122.4915) (layer "B.SilkS")
     (effects (font (size 1.016 1.016) (thickness 0.2032)) (justify mirror))
   )
